Commit message: feat: agregar meta_pkg

File: kalman_description/urdf/xacro/chassis.xacro (robot description, xacro)
@@ -14,5 +14,5 @@
                 <origin xyz="0 0 0" rpy="0 0 0"/>
                 <geometry>
-                    <mesh filename="file://$(find kalman_description)/meshes/carcasa.stl" scale="0.001 0.001 0.001"/>
+                    <mesh filename="package://kalman_description/meshes/carcasa.stl" scale="0.001 0.001 0.001"/>
                 </geometry>
                 <material name="steel"/>
@@ -42,5 +42,5 @@
                 <origin xyz="0 0 0" rpy="0 0 0"/>
                 <geometry>
-                    <mesh filename="file://$(find kalman_description)/meshes/antena.stl" scale="0.001 0.001 0.001"/>
+                    <mesh filename="package://kalman_description/meshes/antena.stl" scale="0.001 0.001 0.001"/>
                 </geometry>
                 <material name="steel"/>
