Commit message: test: prueba de nav2

File: kalman_description/urdf/xacro/caster_wheel.xacro (robot description, xacro)
@@ -8,5 +8,5 @@
                 <origin xyz="0 0 0" rpy="0 0 0"/>
                 <geometry>
-                   <mesh filename="file://$(find kalman_description)/meshes/caster_wheel.stl" scale="0.001 0.001 0.001"/>
+                   <mesh filename="package://kalman_description/meshes/caster_wheel.stl" scale="0.001 0.001 0.001"/>
                 </geometry>
                 <material name="black">
@@ -17,5 +17,5 @@
                 <origin xyz="0 0 0" rpy="0 0 0"/>
                 <!-- <geometry>
-                    <mesh filename="file://$(find kalman_description)/meshes/caster_wheel.stl" scale="0.001 0.001 0.001"/>
+                    <mesh filename="package://kalman_description/meshes/caster_wheel.stl" scale="0.001 0.001 0.001"/>
                 </geometry> -->
                 <geometry>

File: kalman_description/urdf/xacro/wheel.xacro (robot description, xacro)
@@ -11,5 +11,5 @@
                 </geometry-->
                 <geometry>
-                    <mesh filename="file://$(find kalman_description)/meshes/rueda.stl" scale="0.001 0.001 0.001"/>
+                    <mesh filename="package://kalman_description/meshes/rueda.stl" scale="0.001 0.001 0.001"/>
                 </geometry>
                 <material name="black">
